Commit message: Checked and fixed the controller transformations, and fixed the robot message to URDF model mapping
Corrected and fixed the transformations in the Teensy arduino code.
Implemented a sensor_msgs\JointState message from the Teensy Arduino
code and tied it to the URDF model. The robot now uses the
robot_state_controller and the URDF model along with the JointState
messages more extensively.

File: catkin_ws/rot/urdf/rot.urdf (robot description, URDF)
Before this commit: robot RoT, 16 links, 15 joints
Links:
- removed link lidarUnit
- added link lidar; visual box size=0.01 0.035 0.015
- added link ultrasonic_front; visual box size=0.02 0.055 0.03
- added link ultrasonic_rear; visual box size=0.02 0.055 0.03
Joints:
- removed joint lidarUnit_link
- removed joint stearingLeft
- removed joint stearingRight
- added joint jointUltrasonicFront: type fixed, parent base_link, child ultrasonic_front, origin xyz=0.135 0.0 0.0 rpy=0 0 0
- added joint jointUltrasonicRear: type fixed, parent base_link, child ultrasonic_rear, origin xyz=-0.18 0.0 0.05 rpy=0 0 3.14159
- added joint lidar_link: type fixed, parent headBracket3, child lidar, origin xyz=0.052 0.0 0.0 rpy=0 0 0
- added joint steeringLeft: type revolute, parent base_link, child wheelFrontLeft, origin xyz=0.08 0.08 -0.025 rpy=1.5708 0 0, axis 0 1 0, limit lower=-0.349 upper=0.349 effort=100 velocity=1.0
- added joint steeringRight: type revolute, parent base_link, child wheelFrontRight, origin xyz=0.08 -0.08 -0.025 rpy=1.5708 0 0, axis 0 1 0, limit lower=-0.349 upper=0.349 effort=100 velocity=1.0

Commit message: Implemented LIDAR scanning
Implemented the LIDAR scanning function into the Teensy Arduino,
increasedthe Arduino loop frequency from 10Hz to 20Hz and added the
scanning into the URDF model and all associated script including the
Teleop keyboard script.

File: catkin_ws/rot/urdf/rot.urdf (robot description, URDF)
Before this commit: robot RoT, 18 links, 17 joints
Links:
- added link laser_scan; visual box size=0.01 0.035 0.015
Joints:
- added joint laser_scan_link: type fixed, parent base_link, child laser_scan, origin xyz=0.13 0.0 0.13 rpy=0 0 0

Commit message: Implemented point cloud from disparity image
Implemented the point cloud from the disparity image. I had to remove
scalling of the disparity image because it distorts the point cloud. The
scale is not likely to be correct as I had to divide the 3D surface
image from cv2.reprojectImageTo3D to get it close.

File: catkin_ws/rot/urdf/rot.urdf (robot description, URDF)
Before this commit: robot RoT, 19 links, 18 joints
Links:
- added link stereo/pointcloud; visual cylinder length=0.002 radius=0.0025
Joints:
- added joint pointcloud_link: type fixed, parent cameraUnit, child stereo/pointcloud, origin xyz=0.004 -0.035 0.0 rpy=0 1.5708 0

Commit message: Removed pointcloud from urdf
The point cloud wasn't working in the URDF so removed it.

File: catkin_ws/rot/urdf/rot.urdf (robot description, URDF)
Before this commit: robot RoT, 20 links, 19 joints
Links:
- removed link stereo/pointcloud
Joints:
- removed joint pointcloud_link
